File: pcb_design/Monkeys.kicad_pcb (KiCad board)
At the start: 2 copper layers, 144.9 x 59.8 mm, 153 parts, among them IC1 SI4702-C19-GM, J1 JTAG, J2 3.3vSerial, J3 Therm, J4 PJ-320D-4A, J5 10118194-0001LF, Q1 BSS138, Q2 SI2302, Q3 MMBT3904, Q4 MMBT3904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

Commit message: Post Hushcon hardware fixes: - Removed the bad 5v boost converter, inductor and capacitor that resulted in a back-side hardware bypass hack at Hushcon Seattle. - Replaced the over-voltage VDC with +3.3 to the infrared receiver that resulted in a very visible (but kinda cool) wire hack at Hushcon. - Added supplier source links to schematic for battery, battery holder, OLED display and earphones. - Switched the mic amp power and audio path solder bridge jumper to default-on.
Parts:
- removed C10: 10uF, monkeys20221112:C_0603_1608Metric
- removed C11: 100uF, monkeys20221112:CP_EIA-6032-20_AVX-F
- removed L4: 22uH, Inductor_SMD:L_Bourns-SRN4018
- removed U7: Boost5V, Package_TO_SOT_SMD:SOT-23-5
- JP6: footprint Jumper:SolderJumper-2_P1.3mm_Open_RoundedPad1.0x1.5mm -> Jumper:SolderJumper-2_P1.3mm_Bridged_RoundedPad1.0x1.5mm
- turned JP4 to 180 degrees
Connections:
- C40 pad 1: +VDC -> +3V3
- C7 pad 2: +5V -> /AudioAmpPwr
- JP4 pad 1: /EARMIC -> /AMPEDMIC
- JP4 pad 3: /AMPEDMIC -> /EARMIC
- JP6 pad 1: +5V -> /AudioAmpPwr
- R23 pad 1: +5V -> /AudioAmpPwr
- R31 pad 2: +VDC -> +3V3
- SW7 pad 1: Net-(L4-Pad1) -> /AudioAmpPwr
- U4 pad 8: +5V -> /AudioAmpPwr
- U5 pad 4: +VDC -> +3V3
Routing:
- net +5V: track 87.1 -> 0.00 mm, vias 2 -> 0
- net /AudioAmpPwr: track 0.00 -> 85.6 mm, vias 0 -> 2
- net +3V3: track 340.3 -> 351.8 mm, vias 16 -> 18
- net +VDC: track 233.1 -> 225.0 mm
- net Net-(L4-Pad1): track 6.38 -> 0.00 mm
- net Net-(C10-Pad2): track 6.34 -> 0.00 mm
- net GND: track 620.4 -> 616.1 mm
Other:
- board text added: "Audio Amps Switch"
- board text added: "Faxanadu thePhreak Ofir Dilligence"
- board text added: "Monkeybadge 3.8 Designed Jan 2022 - December 2023 By PacketChat, a California Small Corporation"
- board text removed: "Audio Amps 5V"
- board text removed: "Monkeybadge 3.7 Designed Jan 2022 - September 2023 By PacketChat, a California Small Corporation"
