File: pcb_design/Monkeys.kicad_sch (KiCad schematic)
At the start: 156 parts, among them IC1 SI4702-C19-GM, J1 JTAG, J2 3.3vSerial, J3 Therm, J4 PJ-320D-4A, J5 10118194-0001LF, Q1 BSS138, Q2 SI2302, Q3 MMBT3904, Q4 MMBT3904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

Commit message: Post Hushcon hardware fixes: - Removed the bad 5v boost converter, inductor and capacitor that resulted in a back-side hardware bypass hack at Hushcon Seattle. - Replaced the over-voltage VDC with +3.3 to the infrared receiver that resulted in a very visible (but kinda cool) wire hack at Hushcon. - Added supplier source links to schematic for battery, battery holder, OLED display and earphones. - Switched the mic amp power and audio path solder bridge jumper to default-on.
Parts:
- removed C10: 10uF, monkeys20221112:C_0603_1608Metric, symbol Device:C_Small
- removed C11: 100uF, monkeys20221112:CP_EIA-6032-20_AVX-F, symbol Device:C_Polarized_Small
- removed L4: 22uH, Inductor_SMD:L_Bourns-SRN4018, symbol Device:L_Ferrite
- removed U7: Boost5V, Package_TO_SOT_SMD:SOT-23-5, symbol JTFooties2:ME2188C33M5
- JP6: footprint Jumper:SolderJumper-2_P1.3mm_Open_RoundedPad1.0x1.5mm -> Jumper:SolderJumper-2_P1.3mm_Bridged_RoundedPad1.0x1.5mm; symbol Jumper:SolderJumper_2_Open -> Jumper:SolderJumper_2_Bridged
Connections:
- net +5V is gone; now on net AudioAmpPwr: C7.2, JP6.1 (A), R23.1, U4.8 (V+)
- net +3V3: now also C40.1, R31.2, U5.4 (VCC)
- net +VDC: no longer C40.1, R31.2, U5.4 (VCC)
- net AMPEDMIC: now also JP4.1 (A); no longer JP4.3 (B)
- net EARMIC: now also JP4.3 (B); no longer JP4.1 (A)
- net AudioAmpPwr: now reaches SW7.1 (ON)
Other:
- note added: ""Wish this receiver had a buffer." - Ofir"
- note added: "Battery Holder Source:"
- note added: "Battery Source: Shuyang Xinneng Battery Co., Ltd. Hanwang Road And Qiangong Road Intersection North Of 50 Meters, Hanshen Street, Suqian, Jiangsu, China"
- note added: "Earphone Source: Shenzhen Hengxingyuan Technology Co., Ltd. https://www.alibaba.com/product-detail/Custom-Colorful-wired-noise-canceling-earphones_1600397078764.html"
- note added: "OLED Disaplay Source: https://www.aliexpress.us/item/2251832644208699.html"
- note added: "https://www.alibaba.com/product-detail/Factory-direct-high-quality-rechargeable-Li_1600904629787.html"
- note added: "https://www.aliexpress.us/item/3256801509575357.html"
- note removed: "Possible Battery Options"
- note removed: "https://www.alibaba.com/product-detail/14500-3-2V-600mAh-Rechargeable-LiFePO4_60682661392.html?spm=a2700.galleryofferlist.normal_offer.d_title.54bb4347xOxY1X"
- note removed: "https://www.alibaba.com/product-detail/14500-AA-3-7V-800mAh-lithium_62303109893.html?spm=a2700.galleryofferlist.normal_offer.d_title.54bb4347xOxY1X"
- note removed: "https://www.alibaba.com/product-detail/14500-Rechargeable-Battery-AA-2800mAh-3_1600779695589.html?spm=a2700.galleryofferlist.normal_offer.d_title.a7ed2679IqySss"
- note removed: "https://www.alibaba.com/product-detail/14500-lithium-rechargeable-battery-3-7V_62378239464.html?spm=a2700.galleryofferlist.normal_offer.d_title.54bb4347xOxY1X"
- note removed: "https://www.alibaba.com/product-detail/3-7V-800mAh-Li-14500-lithium_1600168392149.html?spm=a2700.galleryofferlist.normal_offer.d_title.54bb4347xOxY1X"
- note removed: "https://www.alibaba.com/product-detail/Cylindrical-14500-3-7V-1200-mAh_1600455662455.html?spm=a2700.galleryofferlist.normal_offer.d_title.54bb4347xOxY1X"
- note removed: "https://www.alibaba.com/product-detail/Energy-Storage-Lithium-Battery-Solar-Home_1600305740461.html?spm=a2700.galleryofferlist.normal_offer.d_title.40e6337bgQTIls"
- note removed: "https://www.alibaba.com/product-detail/Gaonengmax-3-7V-14500-1200mah-li_1600451606725.html?spm=a2700.galleryofferlist.normal_offer.d_title.1a322679m4llBO"
- note removed: "https://www.alibaba.com/product-detail/Rechargeable-Cylinder-14500-1200mAh-Lithium-Battery_1600453629274.html?spm=a2700.galleryofferlist.normal_offer.d_title.1a322679m4llBO"
- note removed: "https://www.alibaba.com/product-detail/SAFD-Lifepo4-Lithium-Ion-Battery-US_1600524362861.html?spm=a2700.galleryofferlist.normal_offer.d_title.40e6337bgQTIls"
